File: Moisture_Sensor.kicad_pcb (KiCad board)
At the start: 2 copper layers, 24 x 19 mm, 17 parts, among them J1 UPDI, J2 OLED SSD1306 0.96in, J3 SOIL SENSOR v1.2, J5 BATTERY 3xAAA, Q1 DMG3415U, SW1 READ BUTTON, U1 ATtiny1614-SSNR, U2 TPS22917DBVR

Commit message: Added name on board back silkscreen
Other:
- board text added: "MOHAMAD DASUKI Rev 1.0.0"
