File: Moisture_Sensor.kicad_pcb (KiCad board)
At the start: 2 copper layers, 24 x 19 mm, 17 parts, among them J1 UPDI, J2 OLED SSD1306 0.96in, J3 SOIL SENSOR v1.2, J5 BATTERY 3xAAA, Q1 DMG3415U, SW1 READ BUTTON, U1 ATtiny1614-SSNR, U2 TPS22917DBVR

Commit message: JLCPCB BOM with LCSC part numbers; switch to JLC basic-library parts
- Add LCSC field to all placed parts (schematic + PCB)
- Passives -> JLC basic equivalents (C1/C4 now 25V), Q1 DMG3415U -> AO3401A (pin-compatible, basic)
- tools/gen_cpl.py now also writes fab/BOM_JLCPCB.csv

Co-authored-by: Copilot App <223556219+Copilot@users.noreply.github.com>
Parts:
- C1: value 10uF 10V X5R -> 10uF 25V X5R
- C4: value 22uF 10V X5R -> 22uF 25V X5R
- Q1: value DMG3415U -> AO3401A
Changed lines of the file:
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@@
 			)
 		)
-		(property "MPN" "RC0603FR-0710KL"
+		(property "MPN" "0603WAF1002T5E"
 			(at 0 0 90)
 			(layer "F.SilkS")
@@
 			)
 		)
-		(property "Manufacturer" "Yageo"
+		(property "Manufacturer" "UNI-ROYAL"
 			(at 0 0 90)
 			(layer "F.SilkS")
@@
 			)
 		)
+		(property "LCSC" "C25804"
+			(at 0 0 0)
+			(layer "F.Fab")
+			(hide yes)
+			(effects
+				(font
+					(size 1.27 1.27)
+				)
+			)
+		)
 		(attr smd)
 		(duplicate_pad_numbers_are_jumpers no)
@@
 			)
 		)
-		(property "MPN" "RC0603FR-0710KL"
+		(property "MPN" "0603WAF1002T5E"
 			(at 0 0 90)
 			(layer "F.SilkS")
@@
 			)
 		)
-		(property "Manufacturer" "Yageo"
+		(property "Manufacturer" "UNI-ROYAL"
 			(at 0 0 90)
 			(layer "F.SilkS")
@@
 			)
 		)
+		(property "LCSC" "C25804"
+			(at 0 0 0)
+			(layer "F.Fab")
+			(hide yes)
+			(effects
+				(font
+					(size 1.27 1.27)
+				)
+			)
+		)
 		(attr smd)
 		(duplicate_pad_numbers_are_jumpers no)
@@
 			)
 		)
-		(property "MPN" "RC0603JR-070RL"
+		(property "MPN" "0603WAF0000T5E"
 			(at 0 0 90)
 			(layer "F.SilkS")
@@
 			)
 		)
-		(property "Manufacturer" "Yageo"
+		(property "Manufacturer" "UNI-ROYAL"
 			(at 0 0 90)
 			(layer "F.SilkS")
@@
 			)
 		)
+		(property "LCSC" "C21189"
+			(at 0 0 0)
+			(layer "F.Fab")
+			(hide yes)
+			(effects
+				(font
+					(size 1.27 1.27)
+				)
+			)
+		)
 		(attr smd)
 		(duplicate_pad_numbers_are_jumpers no)
@@
 			)
 		)
-		(property "Value" "DMG3415U"
+		(property "Value" "AO3401A"
 			(at 0 2.4 0)
 			(layer "F.Fab")
@@
 			)
 		)
-		(property "MPN" "DMG3415U-7"
+		(property "MPN" "AO3401A"
 			(at 0 0 0)
 			(layer "F.SilkS")
@@
 			)
 		)
-		(property "Manufacturer" "Diodes Inc"
+		(property "Manufacturer" "Alpha & Omega"
 			(at 0 0 0)
 			(layer "F.SilkS")
@@
 			)
 		)
+		(property "LCSC" "C15127"
+			(at 0 0 0)
+			(layer "F.Fab")
+			(hide yes)
+			(effects
+				(font
+					(size 1.27 1.27)
+				)
+			)
+		)
 		(attr smd)
 		(duplicate_pad_numbers_are_jumpers no)
@@
 			)
 		)
+		(property "LCSC" "C131337"
+			(at 0 0 0)
+			(layer "F.Fab")
+			(hide yes)
+			(effects
+				(font
+					(size 1.27 1.27)
+				)
+			)
+		)
 		(zone_connect 1)
 		(attr through_hole)
@@
 			)
 		)
+		(property "LCSC" "C2681320"
+			(at 0 0 0)
+			(layer "F.Fab")
+			(hide yes)
+			(effects
+				(font
+					(size 1.27 1.27)
+				)
+			)
+		)
 		(attr smd)
 		(duplicate_pad_numbers_are_jumpers no)
@@
 			)
 		)
-		(property "MPN" "CL10B104KB8NNNC"
+		(property "MPN" "CC0603KRX7R9BB104"
 			(at 0 0 90)
 			(layer "F.SilkS")
@@
 			)
 		)
-		(property "Manufacturer" "Samsung"
+		(property "Manufacturer" "Yageo"
 			(at 0 0 90)
 			(layer "F.SilkS")
@@
 			)
 		)
+		(property "LCSC" "C14663"
+			(at 0 0 0)
+			(layer "F.Fab")
+			(hide yes)
+			(effects
+				(font
+					(size 1.27 1.27)
+				)
+			)
+		)
 		(attr smd)
 		(duplicate_pad_numbers_are_jumpers no)
@@
 			)
 		)
-		(property "MPN" "CL10B104KB8NNNC"
+		(property "MPN" "CC0603KRX7R9BB104"
 			(at 0 0 90)
 			(layer "F.SilkS")
@@
 			)
 		)
-		(property "Manufacturer" "Samsung"
+		(property "Manufacturer" "Yageo"
 			(at 0 0 90)
 			(layer "F.SilkS")
@@
 			)
 		)
+		(property "LCSC" "C14663"
+			(at 0 0 0)
+			(layer "F.Fab")
+			(hide yes)
+			(effects
+				(font
+					(size 1.27 1.27)
+				)
+			)
+		)
 		(attr smd)
 		(duplicate_pad_numbers_are_jumpers no)
@@
 			)
 		)
+		(property "LCSC" "C1588"
+			(at 0 0 0)
+			(layer "F.Fab")
+			(hide yes)
+			(effects
+				(font
+					(size 1.27 1.27)
+				)
+			)
+		)
 		(attr smd)
 		(duplicate_pad_numbers_are_jumpers no)
@@
 			)
 		)
-		(property "MPN" "CL10B104KB8NNNC"
+		(property "MPN" "CC0603KRX7R9BB104"
 			(at 0 0 90)
 			(layer "F.SilkS")
@@
 			)
 		)
-		(property "Manufacturer" "Samsung"
+		(property "Manufacturer" "Yageo"
 			(at 0 0 90)
 			(layer "F.SilkS")
@@
 			)
 		)
+		(property "LCSC" "C14663"
+			(at 0 0 0)
+			(layer "F.Fab")
+			(hide yes)
+			(effects
+				(font
+					(size 1.27 1.27)
+				)
+			)
+		)
 		(attr smd)
 		(duplicate_pad_numbers_are_jumpers no)
@@
 			)
 		)
+		(property "LCSC" "C481364"
+			(at 0 0 0)
+			(layer "F.Fab")
+			(hide yes)
+			(effects
+				(font
+					(size 1.27 1.27)
+				)
+			)
+		)
 		(attr smd)
 		(duplicate_pad_numbers_are_jumpers no)
@@
 			)
 		)
-		(property "Value" "22uF 10V X5R"
+		(property "Value" "22uF 25V X5R"
 			(at 0 1.68 90)
 			(layer "F.Fab")
@@
 			)
 		)
-		(property "MPN" "CL21A226MPQNNNE"
+		(property "MPN" "CL21A226MAQNNNE"
 			(at 0 0 90)
 			(layer "F.SilkS")
@@
 			)
 		)
+		(property "LCSC" "C45783"
+			(at 0 0 0)
+			(layer "F.Fab")
+			(hide yes)
+			(effects
+				(font
+					(size 1.27 1.27)
+				)
+			)
+		)
 		(attr smd)
 		(duplicate_pad_numbers_are_jumpers no)
@@
 			)
 		)
-		(property "Value" "10uF 10V X5R"
+		(property "Value" "10uF 25V X5R"
 			(at 0 1.68 90)
 			(layer "F.Fab")
@@
 			)
 		)
-		(property "MPN" "CL21A106KPFNNNE"
+		(property "MPN" "CL21A106KAYNNNE"
 			(at 0 0 90)
 			(layer "F.SilkS")
@@
 				)
 			)
+		)
+		(property "LCSC" "C15850"
+			(at 0 0 0)
+			(layer "F.Fab")
+			(hide yes)
+			(effects
+				(font
+					(size 1.27 1.27)
+				)
+			)

Commit message: Reroute PCB for 0.2 mm min track / 0.5 mm edge clearance; battery leads soldered to J5 pads
- J5 JST-PH replaced by 2x 2.54 mm TH wire pads (B+/B- silk), removed from JLC BOM/CPL
- gen_pcb: inset router outline for edge clearance, router clearance margin, widen necked tracks,
  solid GND connection on wire pads, preserve back-silk credit text
- DRC 0 violations / 0 unconnected with schematic parity; enclosure re-checked (0 interferences)

Co-authored-by: Copilot App <223556219+Copilot@users.noreply.github.com>
Parts:
- J5: footprint Connector_JST:JST_PH_B2B-PH-K_1x02_P2.00mm_Vertical -> Connector_PinHeader_2.54mm:PinHeader_1x02_P2.54mm_Vertical
- moved J5 0.80 mm to (102.6, 107.2)
- moved R2 0.10 mm to (123.0, 113.0)
Routing:
- net /SCL: track 31.9 -> 23.6 mm, vias 3 -> 1
- net /VBAT: track 39.0 -> 46.5 mm, vias 0 -> 4
- net /BAT_RAW: track 5.75 -> 12.0 mm
- net /CT: track 21.3 -> 16.2 mm, vias 4 -> 2
- net /UPDI: track 21.1 -> 16.9 mm, vias 1 -> 0
- net /LOAD_EN: track 13.6 -> 9.92 mm, vias 0 -> 2
- net /AOUT: track 14.0 -> 10.4 mm, vias 2 -> 1
- net /GND: track 76.1 -> 79.1 mm, vias 1 -> 0
- net /QOD: track 13.4 -> 16.1 mm
- net /SDA: track 40.2 -> 38.3 mm
- net /BTN: track 12.2 -> 12.7 mm
- net /VSW: track 36.5 -> 36.7 mm, vias 2 -> 4
Other:
- board text added: "B+"
- board text added: "B-"
- board text removed: "BATT +"
